Commit message: retry

File: Go_manipulator_description/urdf/Go_manipulator.urdf (robot description, URDF)
Before this commit: robot Go_manipulator, 10 links, 9 joints
Links:
- removed link base_link
- added link link0, mass 0.8410; collision mesh filename=package://Go_manipulator_description/meshes/arm/base_link.S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; visual mesh filename=package://Go_manipulator_description/meshes/arm/base_link.S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
- link gripper_base: geometry collision mesh filename=package://Go_manipulator_description/meshes/gripper/gripper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; visual mesh filename=package://Go_manipulator_description/meshes/gripper/gripper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
- link gripper_finger1: geometry collision mesh filename=package://Go_manipulator_description/meshes/gripper/gripper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; visual mesh filename=package://Go_manipulator_description/meshes/gripper/gripper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
- link gripper_finger2: geometry collision mesh filename=package://Go_manipulator_description/meshes/gripper/gripper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; visual mesh filename=package://Go_manipulator_description/meshes/gripper/gripper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
- link link1: geometry collision mesh filename=package://Go_manipulator_description/meshes/arm/link1.STL; visual mesh filename=package://Go_manipulator_description/meshes/arm/link1.STL
- link link2: geometry collision mesh filename=package://Go_manipulator_description/meshes/arm/link2.STL; visual mesh filename=package://Go_manipulator_description/meshes/arm/link2.STL
- link link3: geometry collision mesh filename=package://Go_manipulator_description/meshes/arm/link3.STL; visual mesh filename=package://Go_manipulator_description/meshes/arm/link3.STL
- link link4: geometry collision mesh filename=package://Go_manipulator_description/meshes/arm/link4.STL; visual mesh filename=package://Go_manipulator_description/meshes/arm/link4.STL
- link link5: geometry collision mesh filename=package://Go_manipulator_description/meshes/arm/link5.STL; visual mesh filename=package://Go_manipulator_description/meshes/arm/link5.STL
Joints:
- joint joint1: parent base_link -> link0

Commit message: 11.04 tmp

File: Go_manipulator_description/urdf/Go_manipulator.urdf (robot description, URDF)
Before this commit: robot Go_manipulator, 10 links, 9 joints
Links:
- link gripper_base: geometry collision mesh filename=package://Go_manipulator_description/meshes/gripper_base.STL; visual mesh filename=package://Go_manipulator_description/meshes/gripper_base.STL
- link gripper_finger1: geometry collision mesh filename=package://Go_manipulator_description/meshes/gripper_finger1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; visual mesh filename=package://Go_manipulator_description/meshes/gripper_finger1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
- link gripper_finger2: geometry collision mesh filename=package://Go_manipulator_description/meshes/gripper_finger2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; visual mesh filename=package://Go_manipulator_description/meshes/gripper_finger2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
- link link0: geometry collision mesh filename=package://Go_manipulator_description/meshes/base_link.STL; visual mesh filename=package://Go_manipulator_description/meshes/base_link.STL
- link link1: geometry collision mesh filename=package://Go_manipulator_description/meshes/link1.STL; visual mesh filename=package://Go_manipulator_description/meshes/link1.STL
- link link2: geometry collision mesh filename=package://Go_manipulator_description/meshes/link2.STL; visual mesh filename=package://Go_manipulator_description/meshes/link2.STL
- link link3: geometry collision mesh filename=package://Go_manipulator_description/meshes/link3.STL; visual mesh filename=package://Go_manipulator_description/meshes/link3.STL
- link link4: geometry collision mesh filename=package://Go_manipulator_description/meshes/link4.STL; visual mesh filename=package://Go_manipulator_description/meshes/link4.STL
- link link5: geometry collision mesh filename=package://Go_manipulator_description/meshes/link5.STL; visual mesh filename=package://Go_manipulator_description/meshes/link5.STL

File: Go_manipulator_description/urdf/go_gripper.urdf.xacro (robot description, xacro)
@@ -1,87 +1,91 @@
 <?xml version="1.0"?>
-<!-- go_gripper.urdf.xacro -->
-<robot xmlns:xacro="http://www.ros.org/wiki/xacro">
-  <xacro:macro name="go_gripper" params="prefix">
-    <xacro:property
-      name="meshes_file_direction"
-      value="package://Go_manipulator_description/meshes"/>
-    <!-- Gripper Base -->
-    <link name="${prefix}gripper_base">
-      <visual>
-        <origin xyz="0 0 0" rpy="0 0 0"/>
-        <geometry>
-          <mesh filename="${meshes_file_direction}/gripper_base.STL"/>
-        </geometry>
-        <material name="grey"/>
-      </visual>
-      <collision>
-        <origin xyz="0 0 0" rpy="0 0 0"/>
-        <geometry>
-          <mesh filename="${meshes_file_direction}/gripper_base.STL"/>
-        </geometry>
-      </collision>
-      <inertial>
-        <origin xyz="0.0001 -0.0283 0" rpy="0 0 0"/>
-        <mass value="0.0568"/>
-        <inertia ixx="3.21e-5" ixy="8.06e-8" ixz="-3.23e-7" iyy="2.21e-5" iyz="-6.81e-18" izz="1.67e-5"/>
-      </inertial>
-    </link>
-    <!-- Gripper Finger 1 and Joint 7 -->
-    <joint name="${prefix}joint7" type="revolute">
-      <parent link="${prefix}gripper_base"/>
-      <child link="${prefix}gripper_finger1"/>
-      <origin xyz="-0.0509 0.0241 -0.0024" rpy="0 0 0"/>
-      <axis xyz="1 0 0"/>
-      <limit lower="-0.2" upper="0.2" effort="100" velocity="0.1"/>
-    </joint>
-    <link name="${prefix}gripper_finger1">
-      <visual>
-        <origin xyz="0 0 0" rpy="0 0 0"/>
-        <geometry>
-          <mesh filename="${meshes_file_direction}/gripper_finger1.STL"/>
-        </geometry>
-        <material name="grey"/>
-      </visual>
-      <collision>
-        <origin xyz="0 0 0" rpy="0 0 0"/>
-        <geometry>
-          <mesh filename="${meshes_file_direction}/gripper_finger1.STL"/>
-        </geometry>
-      </collision>
-      <inertial>
-        <origin xyz="0.0518 -0.0832 -0.0127" rpy="0 0 0"/>
-        <mass value="0.0356"/>
-        <inertia ixx="4.53e-5" ixy="-4.95e-7" ixz="-2.13e-7" iyy="2.41e-5" iyz="-8.24e-6" izz="2.56e-5"/>
-      </inertial>
-    </link>
-    <!-- Gripper Finger 2 and Joint 8 (Mimic Joint) -->
-    <joint name="${prefix}joint8" type="revolute">
-      <parent link="${prefix}gripper_base"/>
-      <child link="${prefix}gripper_finger2"/>
-      <origin xyz="0.0509 0.0241 0.0019" rpy="0 0 3.1416"/>
-      <axis xyz="1 0 0"/>
-      <mimic joint="${prefix}joint7"/>
-      <limit lower="-0.2" upper="0.2" effort="100" velocity="0.1"/>
-    </joint>
-    <link name="${prefix}gripper_finger2">
-      <visual>
-        <origin xyz="0 0 0" rpy="0 0 0"/>
-        <geometry>
-          <mesh filename="${meshes_file_direction}/gripper_finger2.STL"/>
-        </geometry>
-        <material name="grey"/>
-      </visual>
-      <collision>
-        <origin xyz="0 0 0" rpy="0 0 0"/>
-        <geometry>
-          <mesh filename="${meshes_file_direction}/gripper_finger2.STL"/>
-        </geometry>
-      </collision>
-      <inertial>
-        <origin xyz="0.0518 0.0832 0.0141" rpy="0 0 0"/>
-        <mass value="0.0356"/>
-        <inertia ixx="4.53e-5" ixy="4.98e-7" ixz="2.22e-7" iyy="2.41e-5" iyz="-8.25e-6" izz="2.56e-5"/>
-      </inertial>
-    </link>
-  </xacro:macro>
+<robot xmlns:xacro="http://www.ros.org/wiki/xacro" name="go_gripper">
+  <!-- Gripper Base -->
+  <link name="gripper_base">
+    <inertial>
+      <origin xyz="0.0001 -0.0283 0" rpy="0 0 0" />
+      <mass value="0.0568" />
+      <inertia ixx="3.21e-5" ixy="8.06e-8" ixz="-3.23e-7" iyy="2.21e-5" iyz="-6.81e-18" izz="1.67e-5" />
+    </inertial>
+    <visual>
+      <origin xyz="0 0 0" rpy="0 0 0" />
+      <geometry>
+        <mesh filename="package://Go_manipulator_description/meshes/gripper_base.STL" />
+      </geometry>
+      <material name="white"/>
+    </visual>
+    <collision>
+      <origin xyz="0 0 0" rpy="0 0 0" />
+      <geometry>
+        <mesh filename="package://Go_manipulator_description/meshes/gripper_base.STL" />
+      </geometry>
+    </collision>
+  </link>
+  <!-- Joint 6 -->
+  <joint name="joint6" type="revolute">
+    <origin xyz="0.0006 -0.1363 -0.0005" rpy="0 1.5708 0" />
+    <parent link="link5" />
+    <child link="gripper_base" />
+    <axis xyz="0 1 0" />
+    <limit lower="-3.14159" upper="3.14159" effort="1" velocity="1.0" />
+  </joint>
+  <!-- Gripper Finger 1 -->
+  <link name="gripper_finger1">
+    <inertial>
+      <origin xyz="0.0518 -0.0832 -0.0127" rpy="0 0 0" />
+      <mass value="0.0356" />
+      <inertia ixx="4.53e-5" ixy="-4.95e-7" ixz="-2.13e-7" iyy="2.41e-5" iyz="-8.24e-6" izz="2.56e-5" />
+    </inertial>
+    <visual>
+      <origin xyz="0 0 0" rpy="0 0 0" />
+      <geometry>
+        <mesh filename="package://Go_manipulator_description/meshes/gripper_finger1.STL" />
+      </geometry>
+      <material name="black"/>
+    </visual>
+    <collision>
+      <origin xyz="0 0 0" rpy="0 0 0" />
+      <geometry>
+        <mesh filename="package://Go_manipulator_description/meshes/gripper_finger1.STL" />
+      </geometry>
+    </collision>
+  </link>
+  <!-- Joint 7 -->
+  <joint name="joint7" type="revolute">
+    <origin xyz="-0.0509 0.0241 -0.0024" rpy="0 0 0" />
+    <parent link="gripper_base" />
+    <child link="gripper_finger1" />
+    <axis xyz="1 0 0" />
+    <limit lower="-0.2" upper="0.2" effort="100" velocity="0.1" />
+  </joint>
+  <!-- Gripper Finger 2 -->
+  <link name="gripper_finger2">
+    <inertial>
+      <origin xyz="0.0518 0.0832 0.0141" rpy="0 0 0" />
+      <mass value="0.0356" />
+      <inertia ixx="4.53e-5" ixy="4.98e-7" ixz="2.22e-7" iyy="2.41e-5" iyz="-8.25e-6" izz="2.56e-5" />
+    </inertial>
+    <visual>
+      <origin xyz="0 0 0" rpy="0 0 0" />
+      <geometry>
+        <mesh filename="package://Go_manipulator_description/meshes/gripper_finger2.STL" />
+      </geometry>
+      <material name="black"/>
+    </visual>
+    <collision>
+      <origin xyz="0 0 0" rpy="0 0 0" />
+      <geometry>
+        <mesh filename="package://Go_manipulator_description/meshes/gripper_finger2.STL" />
+      </geometry>
+    </collision>
+  </link>
+  <!-- Joint 8 -->
+  <joint name="joint8" type="revolute">
+    <origin xyz="0.0509 0.0241 0.0019" rpy="0 0 3.1416" />
+    <parent link="gripper_base" />
+    <child link="gripper_finger2" />
+    <axis xyz="1 0 0" />
+    <mimic joint="joint7"/>
+    <limit lower="-0.2" upper="0.2" effort="100" velocity="0.1" />
+  </joint>
 </robot>

File: Go_manipulator_description/urdf/go_manipulator.urdf.xacro (robot description, xacro)
@@ -1,27 +1,20 @@
 <?xml version="1.0"?>
-<robot name="go_manipulator" xmlns:xacro="http://www.ros.org/wiki/xacro">
-  <xacro:arg name="prefix" default="" />
-  <xacro:arg name="use_sim" default="false" />
-  <xacro:arg name="use_fake_hardware" default="false" />
-  <xacro:arg name="fake_sensor_commands" default="false" />
-  <!-- ARM 매크로 포함 -->
+<robot xmlns:xacro="http://www.ros.org/wiki/xacro" name="Go_manipulator">
+  <!-- Material Definitions -->
+  <material name="black">
+    <color rgba="0.0 0.0 0.0 1.0"/>
+  </material>
+  <material name="grey">
+    <color rgba="0.5 0.5 0.5 1.0"/>
+  </material>
+  <material name="white">
+    <color rgba="1.0 1.0 1.0 1.0"/>
+  </material>
+  <material name="red">
+    <color rgba="0.8 0.0 0.0 1.0"/>
+  </material>
+  <!-- Include Arm -->
   <xacro:include filename="$(find Go_manipulator_description)/urdf/go_manipulator_arm.urdf.xacro"/>
-  <!-- GRIPPER 매크로 포함 -->
+  <!-- Include Gripper -->
   <xacro:include filename="$(find Go_manipulator_description)/urdf/go_gripper.urdf.xacro"/>
-  <!-- World -->
-  <link name="world"/>
-  <!-- Used for fixing OpenManipulator-Y -->
-  <joint name="$(arg prefix)world_fixed" type="fixed">
-    <parent link="world"/>
-    <child link="$(arg prefix)link0"/>
-    <origin xyz="0.0 0.0 0.0" rpy="0 0 0"/>
-  </joint>
-  <!-- ARM 끝에 GRIPPER를 고정하는 조인트 -->
-  <joint name="$(arg prefix)gripper_fixed" type="fixed">
-    <parent link="$(arg prefix)link6"/>
-    <child link="$(arg prefix)gripper_base"/>
-    <origin xyz="0.0 -0.2398 -0.0005" rpy="0 0 0"/>
-  </joint>
-  <xacro:go_manipulator prefix="$(arg prefix)"/>
-  <xacro:go_gripper prefix="$(arg prefix)"/>
 </robot>
