Commit message: 11.04 tmp

File: Go_manipulator_description/urdf/go_manipulator_arm.urdf.xacro (robot description, xacro)
@@ -1,194 +1,185 @@
 <?xml version="1.0"?>
-<!-- go_manipulator_arm.urdf.xacro -->
-<robot xmlns:xacro="http://www.ros.org/wiki/xacro">
-  <xacro:macro name="go_manipulator" params="prefix">
-    <xacro:property
-      name="meshes_file_direction"
-      value="package://Go_manipulator_description/meshes"/>
-    <!-- Base Link -->
-    <link name="${prefix}link0">
-      <visual>
-        <origin xyz="0 0 0" rpy="0 0 0"/>
-        <geometry>
-          <mesh filename="${meshes_file_direction}/base_link.STL"/>
-        </geometry>
-        <material name="grey"/>
-      </visual>
-      <collision>
-        <origin xyz="0 0 0" rpy="0 0 0"/>
-        <geometry>
-          <mesh filename="${meshes_file_direction}/base_link.STL"/>
-        </geometry>
-      </collision>
-      <inertial>
-        <origin xyz="-0.0676 -0.0067 0.1811" rpy="0 0 0"/>
-        <mass value="0.8410"/>
-        <inertia ixx="0.0026" ixy="2.8e-13" ixz="-4.3e-13" iyy="0.0044" iyz="-5.1e-7" izz="0.0025"/>
-      </inertial>
-    </link>
-    <!-- Joint 1 and Link 1 -->
-    <joint name="${prefix}joint1" type="revolute">
-      <parent link="${prefix}link0"/>
-      <child link="${prefix}link1"/>
-      <origin xyz="-0.0676 -0.18 0.0207" rpy="1.5708 0 0"/>
-      <axis xyz="0 1 0"/>
-      <limit lower="-3.14159" upper="3.14159" effort="1" velocity="1.0"/>
-    </joint>
-    <link name="${prefix}link1">
-      <visual>
-        <origin xyz="0 0 0" rpy="0 0 0"/>
-        <geometry>
-          <mesh filename="${meshes_file_direction}/link1.STL"/>
-        </geometry>
-        <material name="grey"/>
-      </visual>
-      <collision>
-        <origin xyz="0 0 0" rpy="0 0 0"/>
-        <geometry>
-          <mesh filename="${meshes_file_direction}/link1.STL"/>
-        </geometry>
-      </collision>
-      <inertial>
-        <origin xyz="0 0.0180 0.00005" rpy="0 0 0"/>
-        <mass value="0.4427"/>
-        <inertia ixx="0.0006" ixy="8.3e-21" ixz="-1.2e-13" iyy="0.0013" iyz="-6.98e-7" izz="0.0009"/>
-      </inertial>
-    </link>
-    <!-- Joint 2 and Link 2 -->
-    <joint name="${prefix}joint2" type="revolute">
-      <parent link="${prefix}link1"/>
-      <child link="${prefix}link2"/>
-      <origin xyz="0 0.0605 0.00025" rpy="-1.2461 0 0"/>
-      <axis xyz="1 0 0"/>
-      <limit lower="-3.14159" upper="3.14159" effort="1" velocity="1.0"/>
-    </joint>
-    <link name="${prefix}link2">
-      <visual>
-        <origin xyz="0 0 0" rpy="0 0 0"/>
-        <geometry>
-          <mesh filename="${meshes_file_direction}/link2.STL"/>
-        </geometry>
-        <material name="grey"/>
-      </visual>
-      <collision>
-        <origin xyz="0 0 0" rpy="0 0 0"/>
-        <geometry>
-          <mesh filename="${meshes_file_direction}/link2.STL"/>
-        </geometry>
-      </collision>
-      <inertial>
-        <origin xyz="0 0.0253 0.0751" rpy="0 0 0"/>
-        <mass value="0.4222"/>
-        <inertia ixx="0.0010" ixy="-4.91e-15" ixz="1.65e-15" iyy="0.0027" iyz="-0.00027" izz="0.0020"/>
-      </inertial>
-    </link>
-    <!-- Joint 3 and Link 3 -->
-    <joint name="${prefix}joint3" type="revolute">
-      <parent link="${prefix}link2"/>
-      <child link="${prefix}link3"/>
-      <origin xyz="0 0.0360 0.1070" rpy="0.0142 0 0"/>
-      <axis xyz="1 0 0"/>
-      <limit lower="-3.14159" upper="3.14159" effort="1" velocity="1.0"/>
-    </joint>
-    <link name="${prefix}link3">
-      <visual>
-        <origin xyz="0 0 0" rpy="0 0 0"/>
-        <geometry>
-          <mesh filename="${meshes_file_direction}/link3.STL"/>
-        </geometry>
-        <material name="grey"/>
-      </visual>
-      <collision>
-        <origin xyz="0 0 0" rpy="0 0 0"/>
-        <geometry>
-          <mesh filename="${meshes_file_direction}/link3.STL"/>
-        </geometry>
-      </collision>
-      <inertial>
-        <origin xyz="0.0010 0.0340 0.0946" rpy="0 0 0"/>
-        <mass value="0.3496"/>
-        <inertia ixx="0.0022" ixy="-1.15e-5" ixz="-3.21e-5" iyy="0.0019" iyz="-0.00065" izz="0.00032"/>
-      </inertial>
-    </link>
-    <!-- Joint 4 and Link 4 -->
-    <joint name="${prefix}joint4" type="revolute">
-      <parent link="${prefix}link3"/>
-      <child link="${prefix}link4"/>
-      <origin xyz="0 0.0738 0.2053" rpy="1.5283 0 0"/>
-      <axis xyz="1 0 0"/>
-      <limit lower="-3.14159" upper="3.14159" effort="1" velocity="1.0"/>
-    </joint>
-    <link name="${prefix}link4">
-      <visual>
-        <origin xyz="0 0 0" rpy="0 0 0"/>
-        <geometry>
-          <mesh filename="${meshes_file_direction}/link4.STL"/>
-        </geometry>
-        <material name="grey"/>
-      </visual>
-      <collision>
-        <origin xyz="0 0 0" rpy="0 0 0"/>
-        <geometry>
-          <mesh filename="${meshes_file_direction}/link4.STL"/>
-        </geometry>
-      </collision>
-      <inertial>
-        <origin xyz="-0.0225 0.0259 0.0850" rpy="0 0 0"/>
-        <mass value="0.3143"/>
-        <inertia ixx="0.0018" ixy="7.0e-6" ixz="2.29e-5" iyy="0.0016" iyz="-0.00046" izz="0.00022"/>
-      </inertial>
-    </link>
-    <!-- Joint 5 and Link 5 -->
-    <joint name="${prefix}joint5" type="revolute">
-      <parent link="${prefix}link4"/>
-      <child link="${prefix}link5"/>
-      <origin xyz="0 0.0583 0.1913" rpy="-0.2964 0 0"/>
-      <axis xyz="1 0 0"/>
-      <limit lower="-3.14159" upper="3.14159" effort="1" velocity="1.0"/>
-    </joint>
-    <link name="${prefix}link5">
-      <visual>
-        <origin xyz="0 0 0" rpy="0 0 0"/>
-        <geometry>
-          <mesh filename="${meshes_file_direction}/link5.STL"/>
-        </geometry>
-        <material name="grey"/>
-      </visual>
-      <collision>
-        <origin xyz="0 0 0" rpy="0 0 0"/>
-        <geometry>
-          <mesh filename="${meshes_file_direction}/link5.STL"/>
-        </geometry>
-      </collision>
-      <inertial>
-        <origin xyz="-0.0007 -0.0543 -0.0032" rpy="0 0 0"/>
-        <mass value="0.2388"/>
-        <inertia ixx="0.0006" ixy="2.93e-6" ixz="5.84e-7" iyy="7.49e-5" iyz="-4.25e-5" izz="0.0006"/>
-      </inertial>
-    </link>
-    <!-- End Effector Joint and Link -->
-    <joint name="${prefix}joint6" type="revolute">
-      <parent link="${prefix}link5"/>
-      <child link="${prefix}link6"/>
-      <origin xyz="0 0 0.1145" rpy="0 0 0"/>
-      <axis xyz="0 1 0"/>
-      <limit velocity="4.8" effort="1" lower="-1.57" upper="1.57"/>
-      <dynamics damping="0.1"/>
-    </joint>
-    <link name="${prefix}link6">
-      <visual>
-        <origin xyz="0 0 0" rpy="0 0 0"/>
-        <geometry>
-          <box size="0.01 0.01 0.01"/>
-        </geometry>
-        <material name="grey"/>
-      </visual>
-      <collision>
-        <origin xyz="0 0 0" rpy="0 0 0"/>
-        <geometry>
-          <box size="0.01 0.01 0.01"/>
-        </geometry>
-      </collision>
-    </link>
-  </xacro:macro>
+<robot xmlns:xacro="http://www.ros.org/wiki/xacro" name="go_manipulator_arm">
+  <!-- Base Link -->
+  <link name="link0">
+    <inertial>
+      <origin xyz="-0.0676 -0.0067 0.1811" rpy="0 0 0" />
+      <mass value="0.8410" />
+      <inertia ixx="0.0026" ixy="2.8e-13" ixz="-4.3e-13" iyy="0.0044" iyz="-5.1e-7" izz="0.0025" />
+    </inertial>
+    <visual>
+      <origin xyz="0 0 0" rpy="0 0 0" />
+      <geometry>
+        <mesh filename="package://Go_manipulator_description/meshes/base_link.STL" />
+      </geometry>
+      <material name="grey" />
+    </visual>
+    <collision>
+      <origin xyz="0 0 0" rpy="0 0 0" />
+      <geometry>
+        <mesh filename="package://Go_manipulator_description/meshes/base_link.STL" />
+      </geometry>
+    </collision>
+  </link>
+  <!-- Link 1 -->
+  <link name="link1">
+    <inertial>
+      <origin xyz="0 0.0180 0.00005" rpy="0 0 0" />
+      <mass value="0.4427" />
+      <inertia ixx="0.0006" ixy="8.3e-21" ixz="-1.2e-13" iyy="0.0013" iyz="-6.98e-7" izz="0.0009" />
+    </inertial>
+    <visual>
+      <origin xyz="0 0 0" rpy="0 0 0" />
+      <geometry>
+        <mesh filename="package://Go_manipulator_description/meshes/link1.STL" />
+      </geometry>
+      <material name="white"/>
+    </visual>
+    <collision>
+      <origin xyz="0 0 0" rpy="0 0 0" />
+      <geometry>
+        <mesh filename="package://Go_manipulator_description/meshes/link1.STL" />
+      </geometry>
+    </collision>
+  </link>
+  <!-- Joint 1 -->
+  <joint name="joint1" type="revolute">
+    <origin xyz="-0.0676 -0.18 0.0207" rpy="1.5708 0 0" />
+    <parent link="link0" />
+    <child link="link1" />
+    <axis xyz="0 1 0" />
+    <limit lower="-3.14159" upper="3.14159" effort="1" velocity="1.0" />
+  </joint>
+  <!-- Link 2 -->
+  <link name="link2">
+    <inertial>
+      <origin xyz="0 0.0253 0.0751" rpy="0 0 0" />
+      <mass value="0.4222" />
+      <inertia ixx="0.0010" ixy="-4.91e-15" ixz="1.65e-15" iyy="0.0027" iyz="-0.00027" izz="0.0020" />
+    </inertial>
+    <visual>
+      <origin xyz="0 0 0" rpy="0 0 0" />
+      <geometry>
+        <mesh filename="package://Go_manipulator_description/meshes/link2.STL" />
+      </geometry>
+      <material name="white"/>
+    </visual>
+    <collision>
+      <origin xyz="0 0 0" rpy="0 0 0" />
+      <geometry>
+        <mesh filename="package://Go_manipulator_description/meshes/link2.STL" />
+      </geometry>
+    </collision>
+  </link>
+  <!-- Joint 2 -->
+  <joint name="joint2" type="revolute">
+    <origin xyz="0 0.0605 0.00025" rpy="-1.2461 0 0" />
+    <parent link="link1" />
+    <child link="link2" />
+    <axis xyz="1 0 0" />
+    <limit lower="-3.14159" upper="3.14159" effort="1" velocity="1.0" />
+  </joint>
+  <!-- Link 3 -->
+  <link name="link3">
+    <inertial>
+      <origin xyz="0.0010 0.0340 0.0946" rpy="0 0 0" />
+      <mass value="0.3496" />
+      <inertia ixx="0.0022" ixy="-1.15e-5" ixz="-3.21e-5" iyy="0.0019" iyz="-0.00065" izz="0.00032" />
+    </inertial>
+    <visual>
+      <origin xyz="0 0 0" rpy="0 0 0" />
+      <geometry>
+        <mesh filename="package://Go_manipulator_description/meshes/link3.STL" />
+      </geometry>
+      <material name="white"/>
+    </visual>
+    <collision>
+      <origin xyz="0 0 0" rpy="0 0 0" />
+      <geometry>
+        <mesh filename="package://Go_manipulator_description/meshes/link3.STL" />
+      </geometry>
+    </collision>
+  </link>
+  <!-- Joint 3 -->
+  <joint name="joint3" type="revolute">
+    <origin xyz="0 0.0360 0.1070" rpy="0.0142 0 0" />
+    <parent link="link2" />
+    <child link="link3" />
+    <axis xyz="1 0 0" />
+    <limit lower="-3.14159" upper="3.14159" effort="1" velocity="1.0" />
+  </joint>
+  <!-- Link 4 -->
+  <link name="link4">
+    <inertial>
+      <origin xyz="-0.0225 0.0259 0.0850" rpy="0 0 0" />
+      <mass value="0.3143" />
+      <inertia ixx="0.0018" ixy="7.0e-6" ixz="2.29e-5" iyy="0.0016" iyz="-0.00046" izz="0.00022" />
+    </inertial>
+    <visual>
+      <origin xyz="0 0 0" rpy="0 0 0" />
+      <geometry>
+        <mesh filename="package://Go_manipulator_description/meshes/link4.STL" />
+      </geometry>
+      <material name="white"/>
+    </visual>
+    <collision>
+      <origin xyz="0 0 0" rpy="0 0 0" />
+      <geometry>
+        <mesh filename="package://Go_manipulator_description/meshes/link4.STL" />
+      </geometry>
+    </collision>
+  </link>
+  <!-- Joint 4 -->
+  <joint name="joint4" type="revolute">
+    <origin xyz="0 0.0738 0.2053" rpy="1.5283 0 0" />
+    <parent link="link3" />
+    <child link="link4" />
+    <axis xyz="1 0 0" />
+    <limit lower="-3.14159" upper="3.14159" effort="1" velocity="1.0" />
+  </joint>
+  <!-- Link 5 -->
+  <link name="link5">
+    <inertial>
+      <origin xyz="-0.0007 -0.0543 -0.0032" rpy="0 0 0" />
+      <mass value="0.2388" />
+      <inertia ixx="0.0006" ixy="2.93e-6" ixz="5.84e-7" iyy="7.49e-5" iyz="-4.25e-5" izz="0.0006" />
+    </inertial>
+    <visual>
+      <origin xyz="0 0 0" rpy="0 0 0" />
+      <geometry>
+        <mesh filename="package://Go_manipulator_description/meshes/link5.STL" />
+      </geometry>
+      <material name="white"/>
+    </visual>
+    <collision>
+      <origin xyz="0 0 0" rpy="0 0 0" />
+      <geometry>
+        <mesh filename="package://Go_manipulator_description/meshes/link5.STL" />
+      </geometry>
+    </collision>
+  </link>
+  <!-- Joint 5 -->
+  <joint name="joint5" type="revolute">
+    <origin xyz="0 0.0583 0.1913" rpy="-0.2964 0 0" />
+    <parent link="link4" />
+    <child link="link5" />
+    <axis xyz="1 0 0" />
+    <limit lower="-3.14159" upper="3.14159" effort="1" velocity="1.0" />
+  </joint>
+  <!-- End Effector Joint -->
+  <joint name="end_effector_joint" type="fixed">
+    <parent link="link5"/>
+    <child link="end_effector_link"/>
+    <origin xyz="0.0 -0.288 0.0 " rpy="0 0 0"/>
+  </joint>
+  <!-- End Effector Link -->
+  <link name="end_effector_link">
+    <visual>
+      <origin rpy="0 0 0" xyz="0 0 0"/>
+      <geometry>
+        <box size="0.01 0.01 0.01"/>
+      </geometry>
+      <material name="red"/>
+    </visual>
+  </link>
 </robot>
