Commit message: It's something.

File: Go_manipulator_description/urdf/go_gripper.urdf.xacro (robot description, xacro)
@@ -1,8 +1,6 @@
 <?xml version="1.0"?>
 <robot xmlns:xacro="http://www.ros.org/wiki/xacro">
-  <xacro:macro  name="go_gripper" params="perfix">
-    <xacro:property
-      name="meshes_file_direction"
-      value="package://Go_manipulator_description/meshes"/>
+  <xacro:macro  name="go_gripper" params="prefix">
+    <xacro:property name="meshes_file_direction" value="package://Go_manipulator_description/meshes"/>
     <!-- Gripper Base -->
     <link name="${prefix}gripper_base">
@@ -93,3 +91,4 @@
       <limit lower="-0.2" upper="0.2" effort="100" velocity="0.1" />
     </joint>
+  </xacro:macro>
 </robot>

File: Go_manipulator_description/urdf/go_manipulator.urdf.xacro (robot description, xacro)
@@ -2,4 +2,8 @@
 <robot name="Go_manipulator" xmlns:xacro="http://www.ros.org/wiki/xacro">
   <xacro:arg name="prefix" default="" />
+  <xacro:arg name="use_sim" default="false" />
+  <xacro:arg name="use_fake_hardware" default="false" />
+  <xacro:arg name="fake_sensor_commands" default="false" />
+  <xacro:include filename="$(find Go_manipulator_description)/ros2_control/go_manipulator_y_system.ros2_control.xacro" />
   <!-- Material Definitions -->
   <material name="black">
@@ -15,8 +19,10 @@
     <color rgba="0.8 0.0 0.0 1.0"/>
   </material>
-  <!-- Include Arm -->
+  <!-- Arm 포함 -->
   <xacro:include filename="$(find Go_manipulator_description)/urdf/go_manipulator_arm.urdf.xacro"/>
-  <!-- Include Gripper -->
+  <xacro:go_manipulator_arm prefix="$(arg prefix)"/>
+  <!-- Gripper 포함 -->
   <xacro:include filename="$(find Go_manipulator_description)/urdf/go_gripper.urdf.xacro"/>
+  <xacro:go_gripper prefix="$(arg prefix)"/>
   <!-- World -->
   <link name="world"/>
@@ -28,5 +34,5 @@
   </joint>
   <joint name="$(arg prefix)gripper_fixed" type="fixed">
-    <origin xyz="0.0006 -0.1363 -0.0005" rpy="0 1.5708 0" />
+    <origin xyz="0.0 -0.0 0.0" rpy="0 1.5708 0" />
     <parent link="$(arg prefix)link6"/>
     <axis xyz="0 0 0"/>

File: Go_manipulator_description/urdf/go_manipulator_arm.urdf.xacro (robot description, xacro)
@@ -1,8 +1,7 @@
 <?xml version="1.0"?>
 <robot xmlns:xacro="http://www.ros.org/wiki/xacro">
-  <xacro:name="go_manipulator_arm" params="prefix">
-    <xacro:property
-      name="meshes_file_direction"
-      value="package://Go_manipulator/meshes"/>
+  <!-- Define prefix with a default value if not provided -->
+  <xacro:macro name="go_manipulator_arm" params="prefix">
+    <xacro:property name="meshes_file_direction" value="package://Go_manipulator_description/meshes"/>
     <!-- Base Link -->
     <link name="${prefix}link0">
@@ -219,3 +218,4 @@
       </visual>
     </link>
+  </xacro:macro>
 </robot>
