Commit message: go to bed

File: Go_manipulator_description/urdf/go_manipulator.urdf.xacro (robot description, xacro)
@@ -34,5 +34,5 @@
   </joint>
   <joint name="$(arg prefix)gripper_fixed" type="fixed">
-    <origin xyz="0.0 -0.0 0.0" rpy="0 1.5708 0" />
+    <origin xyz="0.0 -0.0 0.0" rpy="0 0 0" />
     <parent link="$(arg prefix)link6"/>
     <axis xyz="0 0 0"/>

File: Go_manipulator_description/urdf/go_manipulator_arm.urdf.xacro (robot description, xacro)
@@ -206,5 +206,5 @@
       <parent link="${prefix}link6"/>
       <child link="end_effector_link"/>
-      <origin xyz="0.0 -0.288 0.0 " rpy="0 0 0"/>
+      <origin xyz="0.0 -0.1475 0.0 " rpy="0 0 0"/>
     </joint>
     <!-- End Effector Link -->
