Commit message: can build. but not work.

File: Go_manipulator_description/ros2_control/go_manipulator_system.ros2_control.xacro (robot description, xacro)
@@ -1,5 +1,5 @@
 <?xml version="1.0"?>
 <robot xmlns:xacro="http://www.ros.org/wiki/xacro">
-  <xacro:macro name="go_manipulator_y_system" params="name prefix use_sim:=^|false use_fake_hardware:=^|false fake_sensor_commands:=^|false">
+  <xacro:macro name="go_manipulator_system" params="name prefix use_sim:=^|false use_fake_hardware:=^|false fake_sensor_commands:=^|false">
     <ros2_control name="${name}" type="system">
       <xacro:if value="$(arg use_sim)">
@@ -131,5 +131,5 @@
       </joint>
       <joint name="${prefix}gripper_finger2">
-        <param name="mimic">${prefix}rh_r1</param>
+        <param name="mimic">${prefix}gripper_finger1</param>
         <param name="multiplier">1</param>
         <command_interface name="position">

File: Go_manipulator_description/urdf/go_manipulator.urdf.xacro (robot description, xacro)
@@ -5,5 +5,5 @@
   <xacro:arg name="use_fake_hardware" default="false" />
   <xacro:arg name="fake_sensor_commands" default="false" />
-  <xacro:include filename="$(find Go_manipulator_description)/ros2_control/go_manipulator_y_system.ros2_control.xacro" />
+  <xacro:include filename="$(find Go_manipulator_description)/ros2_control/go_manipulator_system.ros2_control.xacro" />
   <!-- Material Definitions -->
   <material name="black">
